Commit message: quadrotor follows waypoints based on true estimates

File: roscopter_sim/xacro/multirotor.urdf.xacro (robot description, xacro)
@@ -44,6 +44,35 @@
     <material>Gazebo/${color}</material>
   </gazebo>
-  <!-- ROSflight SIL Plugin -->
-  <xacro:include filename="$(find rosflight_sim)/xacro/rosflight_sil.xacro"/>
-  <xacro:generic_multirotor namespace="${namespace}" parent_link="${namespace}/base_link"/>
+  <!-- ************************* FORCES AND MOMENTS ********************** -->
+  <xacro:include filename="$(find roscopter_sim)/xacro/multirotor_forces_and_moments.xacro"/>
+  <xacro:multirotor_forces_and_moments_macro
+    namespace="${namespace}"
+    parent_link="${namespace}/base_link"
+    command_topic="command"
+    wind_topic="wind"
+    />
+  <!-- ***************** SENSORS ******************* -->
+  <!-- Ground Truth -->
+  <xacro:include filename="$(find rosflight_plugins)/xacro/odometry_sensor.xacro"/>
+  <xacro:odometry_plugin_macro namespace="${namespace}" parent_link="${namespace}/base_link"/>
+  <!-- IMU -->
+  <xacro:include filename="$(find rosflight_plugins)/xacro/imu.xacro"/>
+  <xacro:imu_plugin_macro namespace="${namespace}" parent_link="${namespace}/base_link"/>
+  <!-- Sonar -->
+  <xacro:include filename="$(find rosflight_plugins)/xacro/sonar.xacro"/>
+  <xacro:Sonar_MB1030
+    namespace="${namespace}"
+    parent_link="${namespace}/base_link"
+    sonar_topic="sonar/data">
+    <origin xyz="0 0 0" rpy="0 1.57 0" />
+  </xacro:Sonar_MB1030>
+  <!-- Barometer -->
+  <xacro:include filename="$(find rosflight_plugins)/xacro/barometer.xacro"/>
+  <xacro:barometer_plugin_macro namespace="${namespace}" parent_link="${namespace}/base_link"/>
+  <!-- Magnetometer -->
+  <xacro:include filename="$(find rosflight_plugins)/xacro/magnetometer.xacro"/>
+  <xacro:magnetometer_plugin_macro namespace="${namespace}" parent_link="${namespace}/base_link"/>
+  <!-- GPS -->
+  <xacro:include filename="$(find rosflight_plugins)/xacro/GPS.xacro"/>
+  <xacro:gps_plugin_macro namespace="${namespace}" parent_link="${namespace}/base_link"/>
 </robot>

File: roscopter_sim/xacro/multirotor_forces_and_moments.xacro (robot description, xacro)
@@ -8,20 +8,22 @@
         namespace="${namespace}"
         parent_link="${namespace}/base_link"
-        wind_speed_topic="gazebo/wind_speed"
-        command_topic="${command_topic}"
-        parent_frame_id="${parent_link}"/>
+        wind_topic="gazebo/wind"
+        command_topic="${command_topic}"/>
     </xacro:macro>
   <!-- Macro to add a generic multirotor forces and moments plugin. -->
   <xacro:macro name="multirotor_forces_and_moments_macro"
     params="
-        namespace parent_link wind_speed_topic command_topic parent_frame_id">
+        namespace
+        parent_link
+        wind_topic
+        command_topic
+        ">
     <!-- plugin -->
     <gazebo>
       <plugin filename="libmultirotor_forces_and_moments_plugin.so" name="multirotor_forces_and_moments">
+        <namespace>${namespace}</namespace>
         <linkName>${parent_link}</linkName>
-        <namespace>${namespace}</namespace>
-        <windSpeedTopic>${wind_speed_topic}</windSpeedTopic>
+        <windTopic>${wind_topic}</windTopic>
         <commandTopic>${command_topic}</commandTopic>
-        <parentFrameId>${parent_frame_id}</parentFrameId>
       </plugin>
     </gazebo>
